File: projet/Kicad/MD_Dumper/MD_Dumper.kicad_pcb (KiCad board)
At the start: 2 copper layers, 5 parts, among them U1 74LS273, U2 74LS273, U3 74LS273

Commit message: Update
Routing:
- net (no net): track 0.00 -> 8.74 mm
- net D1_V: track 350.3 -> 346.8 mm
- net D0_V: track 385.7 -> 382.2 mm
- net D4_V: track 321.9 -> 318.9 mm
- net CLK3: track 96.2 -> 98.7 mm
- net D5_V: track 345.8 -> 343.3 mm
- net D8: track 155.9 -> 153.4 mm
- net A22: track 58.1 -> 55.7 mm
- net D9: track 107.4 -> 105.2 mm
- net D10: track 83.5 -> 81.3 mm
- net A16: track 230.8 -> 232.7 mm
- net D2_V: track 301.3 -> 299.5 mm
- net A15: track 204.3 -> 205.7 mm
- net D11: track 63.3 -> 62.0 mm
- net D3_V: track 273.0 -> 271.8 mm
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
Commit message: Update
Routing:
- net D0_V: track 382.2 -> 378.1 mm
- net A16: track 232.7 -> 235.7 mm
- net A8: track 74.5 -> 72.6 mm
- net A4: track 124.0 -> 125.3 mm
- net A9: track 73.1 -> 71.8 mm
- net CLK1: track 252.2 -> 253.5 mm
- net CLK3: track 98.7 -> 100.0 mm
- net D2_V: track 299.5 -> 298.4 mm
- net D5_V: track 343.3 -> 344.3 mm
- net VCC5: track 409.2 -> 410.1 mm
- net A12: track 123.9 -> 122.9 mm
- net D6_V: track 358.0 -> 358.9 mm
- net A13: track 154.0 -> 153.1 mm
- net D7_V: track 382.1 -> 382.9 mm
- net A7: track 123.0 -> 123.8 mm
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
Commit message: Update
Routing:
- net D7_V: track 382.9 -> 385.6 mm
- net D6_V: track 358.9 -> 361.2 mm
- net D5_V: track 344.3 -> 346.2 mm
- net D4_V: track 318.9 -> 320.3 mm
- net CLK3: track 100.0 -> 98.8 mm
- net A7: track 123.8 -> 124.8 mm
- net VCC5: track 410.1 -> 410.8 mm
- net D12: track 68.7 -> 68.2 mm

Commit message: Update
Routing:
- net D7_V: track 385.6 -> 392.4 mm
- net VCC5: track 410.8 -> 405.8 mm
- net D6_V: track 361.2 -> 365.9 mm
- net D0_V: track 378.1 -> 382.4 mm
- net D5_V: track 346.2 -> 349.9 mm
- net D8: track 153.4 -> 157.1 mm
- net D4_V: track 320.3 -> 323.5 mm
- net CLK1: track 253.5 -> 250.9 mm
- net D1_V: track 346.6 -> 349.2 mm
- net D9: track 105.2 -> 107.0 mm
- net D2_V: track 298.4 -> 299.2 mm
- net D10: track 81.3 -> 81.9 mm
Other:
- board outline added: 160 x 100 mm
